Commit message: Performance improvements

File: problems/manipulator_discrete/model/test_5dof.urdf (robot description, URDF)
Before this commit: robot lbr_iiwa, 6 links, 5 joints
Links:
- added link link5, mass 0.2; collision box size=1 0.15 0.15; visual box size=1 0.15 0.15
Joints:
- added joint joint6: type fixed, parent link5, child end_effector, origin xyz=1 0 0 rpy=0 0 0, axis 0 0 1, limit lower=-3.14159265358979323846 upper=3.14159265358979323846 effort=40 velocity=4.0
- joint joint5: child end_effector -> link5; limit lower=-3.14159265358979323846 upper=3.14159265358979323846 effort=40 velocity=4.0 -> lower=-3.14159265358979323846 upper=3.14159265358979323846 effort=50 velocity=4.0; type fixed -> revolute
